Commit message: weld-gun-x1: detailed procedural visual meshes, true X-gun layout
Visual is now generated by tools/generate_meshes.py (trimesh only, no
booleans): MFDC transformer, servo + ball screw drive, pivot clevis,
tapered forged arms crossing at the pivot, ISO 5821-style electrode caps,
cooling hoses and kickless cable.

Collision stays primitives-only (10 box/cylinder) so the throat opening
survives - verified with a 1.5 mm sheet swept into the throat and with a
self-collision sweep over the full joint range.

Co-Authored-By: Claude Fable 5 <noreply@anthropic.com>

File: weld-gun-x1/urdf/weld-gun-x1.urdf (robot description, URDF)
Before this commit: robot weld_gun_x1, 4 links, 3 joints
Links:
- link body: mass 28 -> 72; geometry collision box size=0.200 0.140 0.135; collision box size=0.215 0.195 0.290
- link electrode_arm: mass 7 -> 13; geometry collision cylinder length=0.024 radius=0.011; collision cylinder length=0.040 radius=0.021
Joints:
- joint electrode_joint: limit lower=0 upper=0.30 effort=200 velocity=2.0 -> lower=0 upper=0.42 effort=2400 velocity=1.2; origin xyz=0.05 0 0.42 -> xyz=0.115 0 0.335
- joint tcp_joint: origin xyz=0.375 0 0.36 -> xyz=0.375 0 0.360

Commit message: weld-gun-x1: dimension to published standards and real machine-class specs
Spot gun vendors publish no dimensional drawings (guns are engineered per
application - checked OBARA, NIMAK, Milco, ARO, Electroweld), so the model is
anchored to what IS published instead of arbitrary numbers:

- electrode caps are now exactly ISO 5821 Type F 16 x 20 (l1=20, R1=40 spherical
  face, 1:10 taper) and the electrode force is the standard's own Fmax for a
  16 mm cap: 4.0 kN (was 4.5 kN, which exceeded it)
- throat depth 220 -> 400 mm, the published standard for X-type guns
- mass/inertia derived from the collision primitives, and verified against the
  FANUC R-2000iC/165F published wrist allowables (J5 940 Nm / 89 kgm2,
  J6 490 Nm / 46 kgm2) - all four pass with margin

Co-Authored-By: Claude Fable 5 <noreply@anthropic.com>

File: weld-gun-x1/urdf/weld-gun-x1.urdf (robot description, URDF)
Before this commit: robot weld_gun_x1, 4 links, 3 joints
Links:
- link body: mass 72 -> 78; geometry collision box size=0.200 0.140 0.135; collision box size=0.215 0.195 0.290
- link electrode_arm: mass 13 -> 17; geometry collision cylinder length=0.020 radius=0.009; collision cylinder length=0.048 radius=0.020
Joints:
- joint electrode_joint: limit lower=0 upper=0.42 effort=2400 velocity=1.2 -> lower=0 upper=0.26 effort=1800 velocity=1.2
- joint tcp_joint: origin xyz=0.375 0 0.360 -> xyz=0.553 0 0.360
