Commit message: biw-sedan: decouple visual from collision, ship a curved skin as coloured glb
Collision has to be a convex compound; visual does not. Splitting them lets the
body carry a real outer skin - tumblehome above the beltline, plan-view taper at
the ends, a beltline that drops to the fender and deck, and a crowned roof. None
of those are convex. Door apertures and wheel arches stay real openings.

Visual goes out as glb (16,052 faces, coloured) because glb carries materials;
the builder normalises it to OBJ+MTL. Collision is unchanged: 49 convex STL.

Co-Authored-By: Claude Fable 5 <noreply@anthropic.com>

File: biw-sedan/urdf/biw-sedan.urdf (robot description, URDF)
Before this commit: robot biw_sedan, 1 links, 0 joints
Links:
- link biw: geometry collision mesh filename=../meshes/collision/a_pillar_l.stl; collision mesh filename=../meshes/collision/a_pillar_r.stl
