Commit message: weld-gun-c1: put the transformer behind the mount
Sitting it at throat height put the mass off the tool axis and made it the first
thing to foul near a weld point. Behind the mount the centre of mass lands
almost on the tool axis and the J6 moment drops from 101 to 23 Nm.

It does not change reach on the BIW flanges - measured identical before and
after - so the C frame surrounding the mouth on three sides is what limits this
gun, not the transformer placement. Recorded that comparison in the README
rather than leaving the impression that a short throat means better access.

Co-Authored-By: Claude Fable 5 <noreply@anthropic.com>

File: weld-gun-c1/urdf/weld-gun-c1.urdf (robot description, URDF)
Before this commit: robot weld_gun_c1, 4 links, 3 joints
Links:
- link body: geometry collision box size=0.07 0.116 0.47; collision box size=0.12 0.034 0.115
