Commit message: Model NIMAK 95.020.516 single-jaw opening from measured pivot

File: nimak-multiframegun/urdf/95-020-516-p3u.urdf (robot description, URDF)
Before this commit: robot 95-020-516-p3u, 15 links, 14 joints
Links:
- added link moving_jaw; collision box size=0.055 0.04 0.53; collision box size=0.09 0.04 0.2
- added link moving_tip
- link body: geometry collision box size=0.055 0.04 0.53; collision box size=0.09 0.04 0.2
Joints:
- added joint jaw_opening: type revolute, parent body, child moving_jaw, origin xyz=-0.0134 0 0.59 rpy=0 0 0, axis 0 1 0, limit lower=0 upper=0.349065850399 velocity=0.2
- added joint moving_tip_joint: type fixed, parent moving_jaw, child moving_tip, origin xyz=0 0 0.7 rpy=0 -1.57079632679 0
