Commit message: Rebuild BX250L and NIMAK reference geometry from official sources

File: kawasaki-bx250l/urdf/bx250l-b001.urdf (robot description, URDF)
Before this commit: robot bx250l-b001, 10 links, 9 joints
Links:
- link base_link: geometry collision box size=0.75 0.875 0.03; collision cylinder length=0.244 radius=0.295
- link link1: geometry collision box size=0.55 0.55 0.4; collision cylinder length=0.07 radius=0.3
- link link2: geometry collision box size=0.2 0.22 0.39; collision box size=0.22 0.25 0.38
- link link3: geometry collision cylinder length=0.292 radius=0.17; collision cylinder length=0.42 radius=0.192
- link link4: geometry collision box size=0.06 0.1 0.35; collision box size=0.06 0.1 0.35
- link link5: geometry collision cylinder length=0.2 radius=0.126; collision cylinder length=0.212 radius=0.116
- link link6: geometry collision cylinder length=0.056 radius=0.1; collision cylinder length=0.11 radius=0.11
- link parallel_arm1: geometry collision box size=0.09 0.17 1.23; visual mesh filename=../meshes/parallel_rod.stl
- link parallel_arm2: geometry collision box size=0.09 0.4 0.43; visual mesh filename=../meshes/carrier_bearing.stl

File: nimak-multiframegun/urdf/95-020-516-p3u.urdf (robot description, URDF)
Before this commit: robot 95-020-516-p3u, 17 links, 16 joints
Links:
- link body: geometry collision box size=0.055 0.04 0.53; collision box size=0.09 0.04 0.2
- link moving_jaw: geometry collision box size=0.055 0.04 0.53; collision box size=0.09 0.04 0.2
