Commit message: Align TCP, outlet frames and collision envelopes with the refined visuals
RG2 / RG6: TCP at the closed-pose centre of the visible boots; box and
pivot-cylinder collisions around every link, so the boots, carriers, arms
and QC are enclosed and no collision pair overlaps in only part of the
stroke. DAIHEN CM-7403 / WB-P352L: torch outlet frames on the visible
connectors; CM-7403 collision follows the new shell inside the published
envelope, WB-P352L adds the lifting eyes. Toyota SAE160 TX / DX: collision
for the centred tiller, console, HMI and stays, beacon, foot pins, top
shrouds and the carriage backrest. Joints, limits, mimic rules and visual
meshes are unchanged. Tests, audits, READMEs, provenance and verification
notes follow the new contract; catalog IDs point at the new revisions.

Co-Authored-By: Claude Opus 5.5 <noreply@anthropic.com>

File: daihen-cm-7403/urdf/daihen-cm-7403.urdf (robot description, URDF)
Before this commit: robot daihen_cm_7403, 3 links, 2 joints
Links:
- link base_link: geometry collision box size=0.174 0.066 0.048; collision box size=0.254 0.087 0.066
Joints:
- joint torch_outlet_joint: origin xyz=0 0.3295 0.2 rpy=-1.57079632679 0 0 -> xyz=0.052 0.3175 0.115 rpy=-1.57079632679 0 0

File: daihen-wb-p352l/urdf/daihen-wb-p352l.urdf (robot description, URDF)
Before this commit: robot daihen_wb_p352l, 3 links, 2 joints
Links:
- link base_link: geometry collision box size=0.032 0.007 0.032; collision box size=0.032 0.007 0.032
Joints:
- joint torch_outlet_joint: origin xyz=-0.06 -0.355 0.3 rpy=0 0 0 -> xyz=0.136 -0.326 0.195 rpy=0 0 0

File: onrobot-rg2/urdf/onrobot-rg2.urdf (robot description, URDF)
Before this commit: robot onrobot_rg2_reference, 15 links, 14 joints
Links:
- link rg2_v2_gripper_bracket: geometry collision box size=0.069 0.034 0.038; collision box size=0.075 0.036 0.039
- link rg2_v2_gripper_finger_1_finger_tip: geometry collision box size=0.0215 0.022 0.0542683563099; visual mesh filename=../meshes/rg2_v2_gripper_finger_1_finger_tip.obj
- link rg2_v2_gripper_finger_1_flex_finger: geometry collision box size=0.0114 0.0202 0.0298; visual mesh filename=../meshes/rg2_v2_gripper_finger_1_flex_finger.obj
- link rg2_v2_gripper_finger_1_moment_arm: geometry collision box size=0.0084 0.003 0.0550009309012; collision box size=0.0084 0.003 0.0550009309012
- link rg2_v2_gripper_finger_1_truss_arm: geometry collision box size=0.0084 0.003 0.0550009309012; collision box size=0.0084 0.003 0.0550009309012
- link rg2_v2_gripper_finger_2_finger_tip: geometry collision box size=0.0215 0.022 0.0542683563099; visual mesh filename=../meshes/rg2_v2_gripper_finger_2_finger_tip.obj
- link rg2_v2_gripper_finger_2_flex_finger: geometry collision box size=0.0114 0.0202 0.0298; visual mesh filename=../meshes/rg2_v2_gripper_finger_2_flex_finger.obj
- link rg2_v2_gripper_finger_2_moment_arm: geometry collision box size=0.0084 0.003 0.0550009309012; collision box size=0.0084 0.003 0.0550009309012
- link rg2_v2_gripper_finger_2_truss_arm: geometry collision box size=0.0084 0.003 0.0550009309012; collision box size=0.0084 0.003 0.0550009309012
Joints:
- joint rg2_v2_gripper_grasp_frame_joint: origin xyz=0 0 0.1591 rpy=0 0 0 -> xyz=0 0 0.1781 rpy=0 0 0

File: onrobot-rg6/urdf/onrobot-rg6.urdf (robot description, URDF)
Before this commit: robot onrobot_rg6_reference, 15 links, 14 joints
Links:
- link rg6_v2_gripper_bracket: geometry collision box size=0.076 0.04 0.04; collision box size=0.082 0.062 0.0561
- link rg6_v2_gripper_finger_1_finger_tip: geometry collision box size=0.026 0.025 0.0704033027929; visual mesh filename=../meshes/rg6_v2_gripper_finger_1_finger_tip.obj
- link rg6_v2_gripper_finger_1_flex_finger: geometry collision box size=0.01315 0.025 0.037; visual mesh filename=../meshes/rg6_v2_gripper_finger_1_flex_finger.obj
- link rg6_v2_gripper_finger_1_moment_arm: geometry collision box size=0.011 0.004 0.0800026612057; collision box size=0.011 0.004 0.0800026612057
- link rg6_v2_gripper_finger_1_truss_arm: geometry collision box size=0.011 0.004 0.0800026612057; collision box size=0.011 0.004 0.0800026612057
- link rg6_v2_gripper_finger_2_finger_tip: geometry collision box size=0.026 0.025 0.0704033027929; visual mesh filename=../meshes/rg6_v2_gripper_finger_2_finger_tip.obj
- link rg6_v2_gripper_finger_2_flex_finger: geometry collision box size=0.01315 0.025 0.037; visual mesh filename=../meshes/rg6_v2_gripper_finger_2_flex_finger.obj
- link rg6_v2_gripper_finger_2_moment_arm: geometry collision box size=0.011 0.004 0.0800026612057; collision box size=0.011 0.004 0.0800026612057
- link rg6_v2_gripper_finger_2_truss_arm: geometry collision box size=0.011 0.004 0.0800026612057; collision box size=0.011 0.004 0.0800026612057
Joints:
- joint rg6_v2_gripper_grasp_frame_joint: origin xyz=0 0 0.212 rpy=0 0 0 -> xyz=0 0 0.2164 rpy=0 0 0

File: toyota-sae160/dx/urdf/toyota-sae160-dx.urdf (robot description, URDF)
Before this commit: robot toyota_sae160_dx_reference, 15 links, 14 joints
Links:
- link base_link: geometry collision box size=0.1151 0.3636 0.0266; collision box size=0.1692 0.361 0.291
- link carriage: geometry collision box size=0.1 0.62 0.612; collision box size=1.25 0.18 0.07
- link mast_outer: geometry collision box size=0.036 0.036 0.427719534275; collision box size=0.036 0.036 0.427719534275

File: toyota-sae160/urdf/toyota-sae160.urdf (robot description, URDF)
Before this commit: robot toyota_sae160_tx_reference, 16 links, 15 joints
Links:
- link base_link: geometry collision box size=0.1151 0.3636 0.0266; collision box size=0.1692 0.361 0.291
- link carriage: geometry collision box size=0.1 0.62 0.686; collision box size=1.25 0.18 0.07
- link mast_outer: geometry collision box size=0.036 0.036 0.427719534275; collision box size=0.036 0.036 0.427719534275
