Commit message: Enclose the KUKA, FANUC, MiR1350 and SAE160 mast visuals in their collisions
KUKA KR 210 L150-2 and FANUC M-410iC/185: boxes and axis cylinders computed
from the drawn parts (castings as slab boxes over their clipped surface)
replace the inherited primitives, which left the visuals up to 505 / 537 mm
outside. Joints, frames, limits and meshes are unchanged. Against the visual
meshes' own self-contact over random poses, the new collisions catch every
real pair and drop the old false contacts.

MiR1350: the top-cover box reaches the side reveals below the deck.

Toyota SAE160 TX / DX: guide-roller boxes, the stages' drawn lower
crossmembers and ears, and the outer foot/head ties where drawn; the
carriage block starts at the drawn plate, so nothing touches the carriage
partway through the lift.

Tests, READMEs, provenance and verification notes follow; public docs name
the catalog build process instead of the builder repository.

Co-Authored-By: Claude Opus 5.5 <noreply@anthropic.com>

File: fanuc-m410ic-185/urdf/fanuc-m410ic-185.urdf (robot description, URDF)
Before this commit: robot fanuc_m410ic_185_reference, 14 links, 13 joints
Links:
- link J1_link: geometry collision box size=0.1802 0.4002 0.2501; collision box size=0.1961 0.0851 0.329
- link J2_link: geometry collision box size=0.0834 0.3242 0.3393; collision box size=0.0853 0.3592 0.3393
- link J3_link: geometry collision box size=0.12 0.52 0.12; collision box size=0.22 0.018 0.13
- link J4_link: geometry collision cylinder length=0.0242 radius=0.1251; visual mesh filename=../meshes/J4_link.obj
- link base_link: geometry collision box size=0.085 0.8898 0.4703; collision box size=0.0851 0.8898 0.4703
- link crank_link: geometry collision box size=0.11 0.1402 0.11; collision box size=0.5772 0.0702 0.2002
- link elbow_link: geometry collision box size=0.0702 0.26 0.0702; collision box size=0.0902 0.1002 0.0902
- link level_lower_link: geometry collision box size=0.06 0.0502 1.2201; visual mesh filename=../meshes/level_lower_link.obj
- link level_upper_link: geometry collision box size=1.3 0.0502 0.06; visual mesh filename=../meshes/level_upper_link.obj
- link rod_link: geometry collision box size=0.1201 0.1001 1.1102; collision box size=0.1928 0.08 1.2221
- link wrist_link: geometry collision box size=0.0902 0.342 0.0902; collision box size=0.12 0.043 0.16

File: kuka-kr210-l150/urdf/kuka-kr210-l150.urdf (robot description, URDF)
Before this commit: robot kuka_kr210_l150_reference, 10 links, 9 joints
Links:
- link base_link: geometry collision box size=0.8982 0.8602 0.0871; collision cylinder length=0.0615 radius=0.3472
- link link_1: geometry collision box size=0.115 0.3002 0.481; collision box size=0.115 0.3002 0.6088
- link link_2: geometry collision box size=0.1581 0.0791 0.2414; collision box size=0.26 0.3061 0.26
- link link_3: geometry collision box size=0.1617 0.2464 0.2706; collision box size=0.1617 0.3221 0.383
- link link_4: geometry collision box size=0.196 0.0222 0.196; collision box size=0.5076 0.0361 0.3035
- link link_5: geometry collision cylinder length=0.1806 radius=0.1021; collision cylinder length=0.2072 radius=0.1041
- link link_6: geometry collision cylinder length=0.0377 radius=0.1003; visual mesh filename=../meshes/link_6.obj

File: mir1350/urdf/mir1350.urdf (robot description, URDF)
Before this commit: robot mir1350_reference, 11 links, 10 joints
Links:
- link top_cover: geometry collision box size=1.35 0.91 0.146; visual mesh filename=../meshes/top_cover.obj

File: toyota-sae160/dx/urdf/toyota-sae160-dx.urdf (robot description, URDF)
Before this commit: robot toyota_sae160_dx_reference, 15 links, 14 joints
Links:
- link carriage: geometry collision box size=0.05 0.62 0.552; collision box size=0.14 0.0625 0.06
- link mast_inner: geometry collision box size=0.01 0.3702 0.03; collision box size=0.047 0.018 0.02
- link mast_outer: geometry collision box size=0.0142 0.64 0.08; collision box size=0.0142 0.64 0.08

File: toyota-sae160/urdf/toyota-sae160.urdf (robot description, URDF)
Before this commit: robot toyota_sae160_tx_reference, 16 links, 15 joints
Links:
- link carriage: geometry collision box size=0.05 0.62 0.626; collision box size=0.14 0.0625 0.06
- link mast_inner: geometry collision box size=0.01 0.3702 0.03; collision box size=0.047 0.018 0.02
- link mast_outer: geometry collision box size=0.0142 0.64 0.08; collision box size=0.0142 0.64 0.08
- link mast_stage1: geometry collision box size=0.01 0.5 0.03; collision box size=0.062 0.018 0.02
