Commit message: Size RG2/RG6 from official STEP measurements; end SAE160 shanks at the fork face
OnRobot RG2 / RG6: the product-page STEP files (303_rg2_tool.step,
301_rg6_tool.step) were read as a measuring instrument only; no STEP,
tessellation, outline trace or derived mesh is committed. Sources, hashes and
readings are in each provenance.json.

- mount is the robot-side Quick Changer tool face (robot flange + 13.6 mm);
  pivots and housing move 13.6 mm (RG2) / 20.0 mm (RG6) towards it
- Housing, bracket, links (one-piece, distal clevis), carriers, standard pads
  and dark cover plates re-authored from the measured sizes in a shared
  builder (visual-geometry.mjs, identical in both packages)
- Joint 0 spaces the bare fingers by the datasheet stroke (110 / 160 mm);
  the upper limit is where the standard pads meet (pads stand 4.45 / 5.0 mm
  proud, 101.1 / 150 mm pad travel); TCP at the pads' centre there:
  205.07 mm (was 217.1) / 251.99 mm (was 272.5)
- Datasheet lengths (datum: top of the robot-side QC, mount + 2.5 mm) agree
  within 0.6 mm; collisions enclose every link visual to 1 um
- Contract hashes, audit gates, model tests, audit reports and renders updated

Toyota SAE160: the fork shanks are 50 mm deep and end at the fork face
(x = 0), the face l2 and the load distance refer to; they stood 10 mm in front
of it. Only the carriage OBJ changes; the carriage enclosure limit drops from
10.1 mm to 3.6 mm (roller axle ends).

Co-Authored-By: Claude Opus 5.5 <noreply@anthropic.com>

File: onrobot-rg2/urdf/onrobot-rg2.urdf (robot description, URDF)
Before this commit: robot onrobot_rg2_reference, 15 links, 14 joints
Links:
- link rg2_v2_gripper_body: geometry collision box size=0.0541 0.0367 0.0151; collision box size=0.0541 0.0367 0.0579
- link rg2_v2_gripper_bracket: geometry collision box size=0.0751 0.0411 0.0521; collision cylinder length=0.0172 radius=0.0355
- link rg2_v2_gripper_finger_1_finger_tip: geometry collision box size=0.0195 0.0116 0.0535; collision cylinder length=0.0198 radius=0.002
- link rg2_v2_gripper_finger_1_moment_arm: geometry collision box size=0.0086 0.02 0.0372; collision box size=0.01 0.02 0.0089
- link rg2_v2_gripper_finger_1_truss_arm: geometry collision box size=0.0031 0.017 0.03; collision box size=0.0056 0.02 0.043
- link rg2_v2_gripper_finger_2_finger_tip: geometry collision box size=0.0195 0.0116 0.0535; collision cylinder length=0.0198 radius=0.002
- link rg2_v2_gripper_finger_2_moment_arm: geometry collision box size=0.0086 0.02 0.0372; collision box size=0.01 0.02 0.0089
- link rg2_v2_gripper_finger_2_truss_arm: geometry collision box size=0.0031 0.017 0.03; collision box size=0.0056 0.02 0.043
Joints:
- joint rg2_v2_gripper_body_joint: origin xyz=0 0 0.039 rpy=0 0 0 -> xyz=0 0 0.0362 rpy=0 0 0
- joint rg2_v2_gripper_finger_1_finger_tip_joint: limit lower=0 upper=1.30524 effort=10 velocity=0.5 -> lower=0 upper=1.2326154780499372 effort=10 velocity=0.5; origin xyz=-0.0256 0 0.04868 rpy=0 0.772 0 -> xyz=-0.0256 0 0.04868 rpy=0 0.783937645046 0
- joint rg2_v2_gripper_finger_1_flex_finger_joint: origin xyz=0.00147849585203 0 0.000868356309929 rpy=0 0 0 -> xyz=0.00945 0 0.0214 rpy=0 0 0
- joint rg2_v2_gripper_finger_1_truss_arm_joint: limit lower=0 upper=1.30524 effort=10 velocity=0.5 -> lower=0 upper=1.2326154780499372 effort=10 velocity=0.5; origin xyz=-0.007678 0 0.103297 rpy=0 -0.772 0 -> xyz=-0.0075 0 0.0925 rpy=0 -0.783937645046 0
- joint rg2_v2_gripper_finger_2_finger_tip_joint: limit lower=0 upper=1.30524 effort=10 velocity=0.5 -> lower=0 upper=1.2326154780499372 effort=10 velocity=0.5; origin xyz=-0.0256 0 0.04868 rpy=0 0.772 0 -> xyz=-0.0256 0 0.04868 rpy=0 0.783937645046 0
- joint rg2_v2_gripper_finger_2_flex_finger_joint: origin xyz=0.00147849585203 0 0.000868356309929 rpy=0 0 0 -> xyz=0.00945 0 0.0214 rpy=0 0 0
- joint rg2_v2_gripper_finger_2_truss_arm_joint: limit lower=0 upper=1.30524 effort=10 velocity=0.5 -> lower=0 upper=1.2326154780499372 effort=10 velocity=0.5; origin xyz=-0.007678 0 0.103297 rpy=0 -0.772 0 -> xyz=-0.0075 0 0.0925 rpy=0 -0.783937645046 0
- joint rg2_v2_gripper_grasp_frame_joint: origin xyz=0 0 0.1781 rpy=0 0 0 -> xyz=0 0 0.168866352435 rpy=0 0 0
- joint rg2_v2_gripper_joint: limit lower=0 upper=1.30524 effort=10 velocity=0.5 -> lower=0 upper=1.2326154780499372 effort=10 velocity=0.5; origin xyz=-0.017178 0 0.086797 rpy=0 -0.772 0 -> xyz=-0.017 0 0.076 rpy=0 -0.783937645046 0
- joint rg2_v2_gripper_mirror_joint: limit lower=0 upper=1.30524 effort=10 velocity=0.5 -> lower=0 upper=1.2326154780499372 effort=10 velocity=0.5; origin xyz=-0.017178 0 0.086797 rpy=0 -0.772 0 -> xyz=-0.017 0 0.076 rpy=0 -0.783937645046 0

File: onrobot-rg6/urdf/onrobot-rg6.urdf (robot description, URDF)
Before this commit: robot onrobot_rg6_reference, 15 links, 14 joints
Links:
- link rg6_v2_gripper_body: geometry collision box size=0.0601 0.0427 0.0161; collision box size=0.0602 0.0427 0.057
- link rg6_v2_gripper_bracket: geometry collision box size=0.0824 0.0451 0.0571; collision cylinder length=0.0172 radius=0.0355
- link rg6_v2_gripper_finger_1_finger_tip: geometry collision box size=0.0259 0.0144 0.0674; collision cylinder length=0.0248 radius=0.0027
- link rg6_v2_gripper_finger_1_moment_arm: geometry collision box size=0.0112 0.025 0.0534; collision box size=0.0126 0.025 0.0157
- link rg6_v2_gripper_finger_1_truss_arm: geometry collision box size=0.0027 0.02 0.042; collision box size=0.007 0.025 0.064
- link rg6_v2_gripper_finger_2_finger_tip: geometry collision box size=0.0259 0.0144 0.0674; collision cylinder length=0.0248 radius=0.0027
- link rg6_v2_gripper_finger_2_moment_arm: geometry collision box size=0.0112 0.025 0.0534; collision box size=0.0126 0.025 0.0157
- link rg6_v2_gripper_finger_2_truss_arm: geometry collision box size=0.0027 0.02 0.042; collision box size=0.007 0.025 0.064
Joints:
- joint rg6_v2_gripper_body_joint: origin xyz=0 0 0.0561 rpy=0 0 0 -> xyz=0 0 0.0392 rpy=0 0 0
- joint rg6_v2_gripper_finger_1_finger_tip_joint: limit lower=0 upper=1.3 effort=10 velocity=0.5 -> lower=0 upper=1.2352262299095726 effort=10 velocity=0.5; origin xyz=-0.05503 0 0.05807 rpy=0 0.49 0 -> xyz=-0.05503 0 0.05807 rpy=0 0.486700298502 0
- joint rg6_v2_gripper_finger_1_flex_finger_joint: origin xyz=0.0098 0 0.0218 rpy=0 0 0 -> xyz=0.0113 0 0.0248 rpy=0 0 0
- joint rg6_v2_gripper_finger_1_truss_arm_joint: limit lower=0 upper=1.3 effort=10 velocity=0.5 -> lower=0 upper=1.2352262299095726 effort=10 velocity=0.5; origin xyz=-0.0105 0 0.1111 rpy=0 -0.49 0 -> xyz=-0.0105 0 0.107992 rpy=0 -0.486700298502 0
- joint rg6_v2_gripper_finger_2_finger_tip_joint: limit lower=0 upper=1.3 effort=10 velocity=0.5 -> lower=0 upper=1.2352262299095726 effort=10 velocity=0.5; origin xyz=-0.05503 0 0.05807 rpy=0 0.49 0 -> xyz=-0.05503 0 0.05807 rpy=0 0.486700298502 0
- joint rg6_v2_gripper_finger_2_flex_finger_joint: origin xyz=0.0098 0 0.0218 rpy=0 0 0 -> xyz=0.0113 0 0.0248 rpy=0 0 0
- joint rg6_v2_gripper_finger_2_truss_arm_joint: limit lower=0 upper=1.3 effort=10 velocity=0.5 -> lower=0 upper=1.2352262299095726 effort=10 velocity=0.5; origin xyz=-0.0105 0 0.1111 rpy=0 -0.49 0 -> xyz=-0.0105 0 0.107992 rpy=0 -0.486700298502 0
- joint rg6_v2_gripper_grasp_frame_joint: origin xyz=0 0 0.2164 rpy=0 0 0 -> xyz=0 0 0.212790661239 rpy=0 0 0
- joint rg6_v2_gripper_joint: limit lower=0 upper=1.3 effort=10 velocity=0.5 -> lower=0 upper=1.2352262299095726 effort=10 velocity=0.5; origin xyz=-0.0238 0 0.088 rpy=0 -0.49 0 -> xyz=-0.0238 0 0.084892 rpy=0 -0.486700298502 0
- joint rg6_v2_gripper_mirror_joint: limit lower=0 upper=1.3 effort=10 velocity=0.5 -> lower=0 upper=1.2352262299095726 effort=10 velocity=0.5; origin xyz=-0.0238 0 0.088 rpy=0 -0.49 0 -> xyz=-0.0238 0 0.084892 rpy=0 -0.486700298502 0
