Commit message: Enclose the Robotiq AX visuals in box collisions around the drawn parts
The refined AX visual (PR #15) kept r1's broad collision proxies, which left
the visual up to 80 mm outside on the base (status lights, pallet sensors,
guide rails, cabinet details) and 55 mm on the carriage (triangular cheeks),
while a full base slab filled the open frame.

- Collisions are now axis-aligned boxes generated from the drawn part groups
  in model.mjs (base 16, carriage 6), rounded outwards to 0.1 mm with a
  float32 tolerance so exact faces stay exact: open frame rails and
  crossmembers with the anchor tabs, mast foot, sensors, mast, guide rails,
  lights, cabinet and isolator; carriage shoes and backplate, the deck and
  cheeks in four slabs along the reach, and the robot plate (top on
  robot_mount)
- Joints, frames, limits, drive settings and meshes are unchanged; only the
  URDF collision elements differ. New test: every visual vertex inside its
  link's boxes to 1 um, the base opening stays open
- Contract hash updated in model.test.mjs and verify_motion.py; motion audit,
  README, provenance and verification updated; catalog ID robotiq/ax/ax10/r2

Co-Authored-By: Claude Opus 5.5 <noreply@anthropic.com>

File: robotiq-ax-series-base/urdf/robotiq-ax-series-base.urdf (robot description, URDF)
Before this commit: robot robotiq_ax_series_base, 3 links, 2 joints
Links:
- link base_link: geometry collision box size=0.0315 0.055 0.0675; collision box size=0.0315 0.055 0.0675
- link carriage: geometry collision box size=0.235 0.1308 0.1045; collision box size=0.235 0.1308 0.1603
